Commit message: new script autonomous mode executing the grasping process, script for forward and inverse kinematics , additionals folder for proper execution

File: urdf/fruit_vehicle_arm.urdf.xacro (robot description, xacro)
@@ -774,5 +774,5 @@
       </material>
     </visual>
-    <collision>
+    <!-- <collision>
       <origin
         xyz="-0.332 -0.3825 -0.054"
@@ -782,5 +782,5 @@
           filename="package://fruit_vehicle_arm/meshes/arm_link4.STL" />
       </geometry>
-    </collision>
+    </collision> -->
   </link>
   <joint
@@ -997,6 +997,6 @@
   <joint name="arm_link2_joint">
       <command_interface name="position">
-          <param name="min">-3.14</param>
-          <param name="max">3.14</param>
+          <param name="min">-1.57</param>
+          <param name="max">1.57</param>
       </command_interface>
       <state_interface name="position"/>
@@ -1005,6 +1005,6 @@
   <joint name="arm_link3_joint">
       <command_interface name="position">
-          <param name="min">-3.14</param>
-          <param name="max">3.14</param>
+          <param name="min">-1.0</param>
+          <param name="max">4.5</param>
       </command_interface>
       <state_interface name="position"/>
@@ -1013,6 +1013,6 @@
   <joint name="arm_link4_joint">
       <command_interface name="position">
-          <param name="min">-3.14</param>
-          <param name="max">3.14</param>
+          <param name="min">-2.5</param>
+          <param name="max">2.5</param>
       </command_interface>
       <state_interface name="position"/>
@@ -1030,5 +1030,5 @@
       <always_on>true</always_on>
       <visualize>true</visualize>
-      <update_rate>10</update_rate>
+      <update_rate>5</update_rate>
       <ray>
         <scan>
